File: sch/MEMS_oscillator.kicad_sch (KiCad schematic)
At the start: 14 parts, among them U1 R-78B3.3-2.0

Commit message: Added some notes
Other:
- note added: "Depending in use of mux on top sheet, BUFFERING MAY BE NEEDED DUE TO LOAD PULL. Loading on CLK-port seems to cause extra heating in SiT5721. Output amplifier probably located near or in heated mems structure."
Changed lines of the file:
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@@
     (stroke (width 0) (type default))
+  )
+  (text "Depending in use of mux on top sheet, \nBUFFERING MAY BE NEEDED DUE TO LOAD PULL. \nLoading on CLK-port seems to cause extra\nheating in SiT5721. Output amplifier probably\nlocated near or in heated mems structure."
+    (at 167.64 99.06 0)
+    (effects (font (size 1.27 1.27)) (justify left bottom))
   )
   (text "Place referece thermally isolated on pcb. \nWith provisions for enclosure to protect\nfrom draught"
