File: sch/mems_ref_osc.kicad_sch (KiCad schematic)
At the start: 7 parts, among them J1 Screw_Terminal_01x02, J2 Conn_Coaxial, J5 Conn_Coaxial

Commit message: Added some notes
Parts:
- removed L1: L, symbol Device:L
- added C18, C19: C, symbol Device:C
- added U3: L7805, symbol Regulator_Linear:L7805
Connections:
- net +5VD: now also C18.1, U3.3 (OUT)
- net GND: now also C18.2, C19.2, U3.2 (GND)
- net +BATT: now reaches C1.1, J1.2 (Pin_2)
- net +BATT: now also C19.1, U3.1 (IN)
Other:
- sheet counters renamed generate_pps
- note added: "Figure out a good use for this mux... And what signals? int_ref, ext_ref, divided?"
- note added: "TODO * DIFF/SE BUFF FOR PPS IN/OUT * Add mux for PPS signals? * Put SiT92216 in a useful place * Add input/output connectors * General clean up for readability"
- note removed: "BUFFERING NEEDED DUE TO LOAD PULL"
- note removed: "TODO * DIFF/SE BUFF FOR PPS IN/OUT * Put SiT92216 in a useful place. * Add input/output connectors * General clean up for readability"
- moved on the sheet: C3, J2, J5, U7
