File: sch/uc_and_if.kicad_sch (KiCad schematic)
At the start: 10 parts, among them J3 Conn_02x02_Top_Bottom, SW1 RotaryEncoder_Switch, SW2 SW_SPDT

Commit message: Added some notes
Connections:
- net at SW2.3 (C): now also J3.4 (Pin_4)
- new net +BATT: J3.3 (Pin_3)
- now unconnected: SW2.1 (A)
Other:
- note added: "1-3 for battery power 2-4 to power via 5v. Arduino can also supply 5V- Do not have usb conected when supplying 5v to arduino"
- moved on the sheet: C10, C9, L3, SW2
